File: bvsys1.brd (EAGLE design)
At the start: 160 x 100 mm, 20 parts

Commit message: Small changes at the office
Parts:
- removed R3: (no value), eagle-ltspice:0204/7
- moved D1 2.00 mm to (54.0, 30.0)
- turned R4 to 180 degrees
Connections:
- removed net N$2: ATTINY84A-PU.1, LCD.3, R3.2, SENS_1.3, SENS_2.3, SENS_3.3, SENS_4.3, U$2.OUT+
- removed net N$20: D1.C, LCD.4, R3.1, R4.1
- new net 5V: ATTINY84A-PU.1, LCD.3, R4.2, SENS_1.3, SENS_2.3, SENS_3.3, SENS_4.3, U$2.OUT+
- new net N$21: D1.C, LCD.4, R4.1
- net GND: no longer R4.2
Routing:
- net 5V: track 0.00 -> 120.0 mm
- net N$2: track 113.6 -> 0.00 mm
- net N$21: track 0.00 -> 18.8 mm
- net N$20: track 8.91 -> 0.00 mm
Changed lines of the file:
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@@
 <attribute name="OC_NEWARK" value="unknown" x="42" y="36" size="3.81" layer="27" rot="R180" display="off"/>
 </element>
-<element name="R3" library="eagle-ltspice" library_urn="urn:adsk.eagle:library:217" package="0204/7" package3d_urn="urn:adsk.eagle:package:13274/1" value="" x="46" y="30" rot="R180">
-<attribute name="SPICEMODEL" value="NONE" x="46" y="30" size="1.778" layer="27" rot="R180" display="off"/>
-<attribute name="SPICEPREFIX" value="R" x="46" y="30" size="1.778" layer="27" rot="R180" display="off"/>
+<element name="R4" library="eagle-ltspice" library_urn="urn:adsk.eagle:library:217" package="0204/7" package3d_urn="urn:adsk.eagle:package:13274/1" value="" x="54" y="34" rot="R180">
+<attribute name="SPICEMODEL" value="NONE" x="54" y="34" size="1.778" layer="27" rot="R180" display="off"/>
+<attribute name="SPICEPREFIX" value="R" x="54" y="34" size="1.778" layer="27" rot="R180" display="off"/>
 </element>
-<element name="R4" library="eagle-ltspice" library_urn="urn:adsk.eagle:library:217" package="0204/7" package3d_urn="urn:adsk.eagle:package:13274/1" value="" x="54" y="34">
-<attribute name="SPICEMODEL" value="NONE" x="54" y="34" size="1.778" layer="27" display="off"/>
-<attribute name="SPICEPREFIX" value="R" x="54" y="34" size="1.778" layer="27" display="off"/>
-</element>
-<element name="D1" library="diode" library_urn="urn:adsk.eagle:library:210" package="DO34Z7" package3d_urn="urn:adsk.eagle:package:43364/1" value="" x="54" y="32"/>
+<element name="D1" library="diode" library_urn="urn:adsk.eagle:library:210" package="DO34Z7" package3d_urn="urn:adsk.eagle:package:43364/1" value="" x="54" y="30"/>
 </elements>
 <signals>
@@
 <contactref element="SENS_3" pad="2"/>
 <contactref element="D4" pad="C"/>
-<wire x1="44" y1="38" x2="46" y2="38" width="0.508" layer="1"/>
-<wire x1="46" y1="38" x2="50" y2="38" width="0.508" layer="1"/>
 <wire x1="60" y1="16" x2="60" y2="10" width="0.508" layer="1"/>
 <wire x1="60" y1="10" x2="60" y2="4" width="0.508" layer="1"/>
-<wire x1="44" y1="38" x2="40" y2="38" width="0.508" layer="1"/>
-<wire x1="40" y1="38" x2="38" y2="38" width="0.508" layer="1"/>
-<wire x1="38" y1="38" x2="18" y2="38" width="0.508" layer="1"/>
-<wire x1="18" y1="38" x2="16.188" y2="39.812" width="0.508" layer="1"/>
-<wire x1="16.188" y1="39.812" x2="16.188" y2="41.364" width="0.508" layer="1"/>
 <wire x1="6.73" y1="41.5" x2="16.052" y2="41.5" width="0.508" layer="1"/>
 <wire x1="16.052" y1="41.5" x2="16.188" y2="41.364" width="0.508" layer="1"/>
-<wire x1="18" y1="38" x2="16.19" y2="38" width="0.508" layer="1"/>
-<wire x1="16.19" y1="38" x2="12" y2="33.81" width="0.508" layer="1"/>
 <wire x1="60" y1="16" x2="60" y2="22" width="0.508" layer="1"/>
 <wire x1="60" y1="22" x2="60" y2="28" width="0.508" layer="1"/>
@@
 <contactref element="LED" pad="1"/>
 <wire x1="40.73" y1="36" x2="40.73" y2="37.27" width="0.508" layer="1"/>
-<wire x1="40.73" y1="37.27" x2="40" y2="38" width="0.508" layer="1"/>
-<wire x1="45.81" y1="36" x2="45.81" y2="37.81" width="0.508" layer="1"/>
-<wire x1="45.81" y1="37.81" x2="46" y2="38" width="0.508" layer="1"/>
-<contactref element="R4" pad="2"/>
-<contactref element="D1" pad="A"/>
 <contactref element="LCD" pad="5"/>
-<wire x1="50" y1="38" x2="56" y2="38" width="0.6096" layer="1"/>
-<wire x1="56" y1="38" x2="58" y2="38" width="0.6096" layer="1"/>
-<wire x1="58" y1="38" x2="60" y2="36" width="0.6096" layer="1"/>
-<wire x1="60" y1="36" x2="60" y2="34" width="0.6096" layer="1"/>
-<wire x1="60" y1="34" x2="60" y2="32" width="0.6096" layer="1"/>
-<wire x1="60" y1="32" x2="60" y2="28" width="0.6096" layer="1"/>
+<wire x1="60" y1="30" x2="60" y2="36" width="0.6096" layer="1"/>
+<wire x1="60" y1="30" x2="60" y2="28" width="0.6096" layer="1"/>
 <wire x1="55.812" y1="41.364" x2="56" y2="41.176" width="0.6096" layer="1"/>
-<wire x1="56" y1="41.176" x2="56" y2="38" width="0.6096" layer="1"/>
 <wire x1="47.81" y1="19.62" x2="50.54" y2="22.35" width="0.6096" layer="1"/>
 <wire x1="50.54" y1="22.35" x2="50.54" y2="26" width="0.6096" layer="1"/>
-<wire x1="57.81" y1="32" x2="57.81" y2="34" width="0.6096" layer="1"/>
-<wire x1="50.54" y1="26" x2="56.54" y2="32" width="0.6096" layer="1"/>
-<wire x1="56.54" y1="32" x2="57.81" y2="32" width="0.6096" layer="1"/>
-<wire x1="57.81" y1="32" x2="60" y2="32" width="0.6096" layer="1"/>
+<contactref element="D1" pad="A"/>
+<wire x1="56" y1="41.176" x2="56" y2="40" width="0.6096" layer="1"/>
+<wire x1="12" y1="33.81" x2="16" y2="37.81" width="0.6096" layer="1"/>
+<wire x1="16" y1="37.81" x2="16" y2="40" width="0.6096" layer="1"/>
+<wire x1="16" y1="40" x2="40" y2="40" width="0.6096" layer="1"/>
+<wire x1="40" y1="40" x2="46" y2="40" width="0.6096" layer="1"/>
+<wire x1="46" y1="40" x2="49.63078125" y2="40" width="0.6096" layer="1"/>
+<wire x1="49.63078125" y1="40" x2="50.07158125" y2="39.5592" width="0.6096" layer="1"/>
+<wire x1="50.07158125" y1="39.5592" x2="52.40841875" y2="39.5592" width="0.6096" layer="1"/>
+<wire x1="52.40841875" y1="39.5592" x2="52.84921875" y2="40" width="0.6096" layer="1"/>
+<wire x1="52.84921875" y1="40" x2="56" y2="40" width="0.6096" layer="1"/>
+<wire x1="40.73" y1="36" x2="40.73" y2="39.27" width="0.6096" layer="1"/>
+<wire x1="40.73" y1="39.27" x2="40" y2="40" width="0.6096" layer="1"/>
+<wire x1="45.81" y1="36" x2="45.81" y2="39.81" width="0.6096" layer="1"/>
+<wire x1="45.81" y1="39.81" x2="46" y2="40" width="0.6096" layer="1"/>
+<wire x1="50.54" y1="26" x2="50.19" y2="26.35" width="0.6096" layer="1"/>
+<wire x1="57.81" y1="30" x2="60" y2="30" width="0.6096" layer="1"/>
+<wire x1="54" y1="30" x2="57.81" y2="30" width="0.6096" layer="1"/>
+<wire x1="50.54" y1="26" x2="50.54" y2="26.54" width="0.6096" layer="1"/>
+<wire x1="50.54" y1="26.54" x2="54" y2="30" width="0.6096" layer="1"/>
+<wire x1="60" y1="36" x2="56" y2="40" width="0.6096" layer="1"/>
+<wire x1="16" y1="40" x2="16.188" y2="41.364" width="0" layer="19" extent="1-1"/>
 </signal>
 <signal name="N$12">
@@
 <wire x1="50.92" y1="9.46" x2="47.81" y2="9.46" width="0.6096" layer="1"/>
 </signal>
-<signal name="N$2">
+<signal name="5V">
 <contactref element="ATTINY84A-PU" pad="1"/>
 <contactref element="LCD" pad="3"/>
@@
 <wire x1="60" y1="40" x2="62.54" y2="37.46" width="0.508" layer="1"/>
 <wire x1="62.54" y1="37.46" x2="62.54" y2="22" width="0.508" layer="1"/>
-<contactref element="R3" pad="2"/>
 <wire x1="62.54" y1="4" x2="62.54" y2="2.54" width="0.6096" layer="1"/>
 <wire x1="62.54" y1="2.54" x2="61.3208" y2="1.3208" width="0.6096" layer="1"/>
 <wire x1="44.6792" y1="1.3208" x2="44" y2="2" width="0.6096" layer="1"/>
-<wire x1="44" y1="2" x2="44" y2="18" width="0.6096" layer="1"/>
+<wire x1="44" y1="2" x2="44" y2="21.62" width="0.6096" layer="1"/>
 <wire x1="42" y1="19.62" x2="40.19" y2="19.62" width="0.6096" layer="1"/>
 <wire x1="61.3208" y1="1.3208" x2="44.6792" y2="1.3208" width="0.6096" layer="1"/>
-<wire x1="42" y1="19.62" x2="44.19" y2="21.81" width="0.6096" layer="1"/>
-<wire x1="44.19" y1="21.81" x2="45.46" y2="23.08" width="0.6096" layer="1"/>
+<wire x1="42" y1="19.62" x2="44" y2="21.62" width="0.6096" layer="1"/>
+<wire x1="44" y1="21.62" x2="45.46" y2="23.08" width="0.6096" layer="1"/>
 <wire x1="45.46" y1="23.08" x2="45.46" y2="26" width="0.6096" layer="1"/>
-<wire x1="44" y1="18" x2="44" y2="21.62" width="0.6096" layer="1"/>
-<wire x1="44" y1="21.62" x2="44.19" y2="21.81" width="0.6096" layer="1"/>
-<wire x1="42.19" y1="30" x2="45.46" y2="26.73" width="0.6096" layer="1"/>
 <wire x1="45.46" y1="26.73" x2="45.46" y2="26" width="0.6096" layer="1"/>
+<contactref element="R4" pad="2"/>
+<wire x1="50.19" y1="34" x2="48" y2="34" width="0.6096" layer="1"/>
+<wire x1="48" y1="34" x2="45.46" y2="31.46" width="0.6096" layer="1"/>
+<wire x1="45.46" y1="31.46" x2="45.46" y2="26" width="0.6096" layer="1"/>
 </signal>
 <signal name="N$4">
@@
 <wire x1="34" y1="35.81" x2="34.19" y2="36" width="0.508" layer="1"/>
 <contactref element="LED" pad="4"/>
-<wire x1="34" y1="35.81" x2="34.19" y2="36" width="0.508" layer="1"/>
 <wire x1="34.19" y1="36" x2="38.19" y2="36" width="0.508" layer="1"/>
 </signal>
@@
 <wire x1="27.23" y1="30.5" x2="28.61" y2="31.88" width="0.508" layer="1"/>
 </signal>
-<signal name="N$20">
-<contactref element="R3" pad="1"/>
+<signal name="N$21">
+<contactref element="LCD" pad="4"/>
+<contactref element="D1" pad="C"/>
 <contactref element="R4" pad="1"/>
-<contactref element="D1" pad="C"/>
-<contactref element="LCD" pad="4"/>
-<wire x1="49.81" y1="30" x2="49.81" y2="29.81" width="0.6096" layer="1"/>
-<wire x1="49.81" y1="29.81" x2="48" y2="28" width="0.6096" layer="1"/>
-<wire x1="48" y1="28" x2="48" y2="26" width="0.6096" layer="1"/>
-<wire x1="49.81" y1="30" x2="50.19" y2="30.38" width="0.6096" layer="1"/>
-<wire x1="50.19" y1="30.38" x2="50.19" y2="32" width="0.6096" layer="1"/>
-<wire x1="50.19" y1="32" x2="50.19" y2="34" width="0.6096" layer="1"/>
+<wire x1="57.81" y1="32" x2="57.81" y2="34" width="0.6096" layer="1"/>
+<wire x1="48" y1="26" x2="48" y2="30" width="0.6096" layer="1"/>
+<wire x1="50.19" y1="30" x2="48" y2="30" width="0.6096" layer="1"/>
+<wire x1="48" y1="30" x2="50" y2="32" width="0.6096" layer="1"/>
+<wire x1="50" y1="32" x2="57.81" y2="32" width="0.6096" layer="1"/>
 </signal>
 </signals>
